Commit message: Arm urdf completed!

File: pkg/src/urdf/Robot.urdf (robot description, URDF)
Before this commit: robot Robot, 8 links, 7 joints
Links:
- link l_Base001: geometry collision box size=0.26 0.192 0.005000000000000001; visual mesh filename=package://urdf_export/meshes/arm_cad_base_kj48jr.dae
- link l_Claw001: geometry collision box size=0.061 0.030000000000000013 0.07; visual mesh filename=package://urdf_export/meshes/arm_cad_claw_15ag4t.dae
- link l_Link006: geometry collision box size=0.12200000000000003 0.151 0.09; visual mesh filename=package://urdf_export/meshes/arm_cad_link0_7pttdh.dae
- link l_Link007: geometry collision box size=0.1025 0.08 0.389984812280998; visual mesh filename=package://urdf_export/meshes/arm_cad_link1_el1qd7.dae
- link l_Link008: geometry collision box size=0.092 0.1 0.25500000000000034; visual mesh filename=package://urdf_export/meshes/arm_cad_link2_zjndgx.dae
- link l_Link009: geometry collision box size=0.075 0.075 0.10748576151343571; visual mesh filename=package://urdf_export/meshes/arm_cad_link3_edo7o8.dae
- link l_Link010: geometry collision box size=0.21919360070894503 0.088 0.07941104040710273; visual mesh filename=package://urdf_export/meshes/arm_cad_link4_rbcbnv.dae
- link l_Link011: geometry collision box size=0.078 0.05000000000000002 0.050000000000000114; visual mesh filename=package://urdf_export/meshes/arm_cad_link5_pga2bj.dae
Joints:
- joint l_Base001__to__l_Link006: limit lower=-3.141592653589793 upper=3.141592653589793 effort=0.0 velocity=0.017453292519943295 -> lower=-3.141592653589793 upper=3.141592653589793 effort=0.0 velocity=3.141592653589793
- joint l_Link006__to__l_Link007: limit lower=-1.5707963267948966 upper=1.5707963267948966 effort=0.0 velocity=0.017453292519943295 -> lower=-1.5707963267948966 upper=1.5707963267948966 effort=0.0 velocity=3.141592653589793
- joint l_Link007__to__l_Link008: limit lower=-1.5707963267948966 upper=1.5707963267948966 effort=0.0 velocity=0.017453292519943295 -> lower=-1.5707963267948966 upper=1.5707963267948966 effort=0.0 velocity=3.141592653589793; origin xyz=0.0 -0.31 0.0925 rpy=-3.141592653589793 0 3.141592653589793 -> xyz=0.0 -0.31 0.0925 rpy=-3.141592653589793 0 3.1415926535897927
- joint l_Link008__to__l_Link009: limit lower=-3.141592653589793 upper=3.141592653589793 effort=0.0 velocity=0.017453292519943295 -> lower=-3.141592653589793 upper=3.141592653589793 effort=0.0 velocity=3.141592653589793
- joint l_Link009__to__l_Link010: limit lower=-3.141592653589793 upper=0.0 effort=0.0 velocity=0.017453292519943295 -> lower=-3.141592653589793 upper=0.0 effort=0.0 velocity=3.141592653589793; origin xyz=0.0375 0.0 -0.07 rpy=-1.570796326794897 0 1.5707963267948966 -> xyz=0.0375 0.0 -0.07 rpy=-1.5707963267948966 0 1.5707963267948963
- joint l_Link010__to__l_Link011: limit lower=-1.5707963267948966 upper=1.5707963267948966 effort=0.0 velocity=0.017453292519943295 -> lower=-1.5707963267948966 upper=1.5707963267948966 effort=0.0 velocity=3.141592653589793
- joint l_Link011__to__l_Claw001: limit lower=-3.141592653589793 upper=3.141592653589793 effort=0.0 velocity=0.017453292519943295 -> lower=-3.141592653589793 upper=3.141592653589793 effort=0.0 velocity=3.141592653589793; origin xyz=-0.025 0.0 -0.039 rpy=3.141592653589793 -1.5707963267948961 0 -> xyz=-0.025 0.0 -0.039 rpy=-3.141592653589793 -1.5707963267948961 0

Commit message: Package name revised

File: pkg/src/urdf/Robot.urdf (robot description, URDF)
Before this commit: robot Robot, 8 links, 7 joints
Links:
- link l_Base001: geometry collision box size=0.26 0.192 0.005000000000000001; visual mesh filename=package://meta_engineer_arm/meshes/arm_cad_base_kj48jr.dae
- link l_Claw001: geometry collision box size=0.061 0.030000000000000013 0.07; visual mesh filename=package://meta_engineer_arm/meshes/arm_cad_claw_15ag4t.dae
- link l_Link006: geometry collision box size=0.12200000000000003 0.151 0.09; visual mesh filename=package://meta_engineer_arm/meshes/arm_cad_link0_7pttdh.dae
- link l_Link007: geometry collision box size=0.1025 0.08 0.389984812280998; visual mesh filename=package://meta_engineer_arm/meshes/arm_cad_link1_el1qd7.dae
- link l_Link008: geometry collision box size=0.092 0.1 0.25500000000000034; visual mesh filename=package://meta_engineer_arm/meshes/arm_cad_link2_zjndgx.dae
- link l_Link009: geometry collision box size=0.075 0.075 0.10748576151343571; visual mesh filename=package://meta_engineer_arm/meshes/arm_cad_link3_edo7o8.dae
- link l_Link010: geometry collision box size=0.21919360070894503 0.088 0.07941104040710273; visual mesh filename=package://meta_engineer_arm/meshes/arm_cad_link4_rbcbnv.dae
- link l_Link011: geometry collision box size=0.078 0.05000000000000002 0.050000000000000114; visual mesh filename=package://meta_engineer_arm/meshes/arm_cad_link5_pga2bj.dae
